Commit message: new robot model finish chassis

File: src/mybot_description/urdf/mybot.xacro (robot description, xacro)
@@ -2,155 +2,27 @@
 <robot name="myrobot" xmlns:xacro="http://www.ros.org/wiki/xacro">
   <xacro:include filename="$(find mybot_description)/urdf/mybot.gazebo" />
-  <xacro:include filename="$(find mybot_description)/urdf/materials.xacro" />
+  <property name="M_PI" value="3.14159" />
+  <property name="M_PI_2" value="3.14159" />
+  <property name="base_mass" value="5" />
+  <property name="base_radius" value="0.15"/>
+  <property name="base_height" value="0.02"/>
   <link name='chassis'>
-    <pose>0 0 0.1 0 0 0</pose>
     <inertial>
-      <mass value="10.0"/>
-      <origin xyz="0.0 0 0.1" rpy=" 0 0 0"/>
-      <inertia
-          ixx="0.5" ixy="0" ixz="0"
-          iyy="1" iyz="0"
-          izz="0.1"
-      />
+      <mass value="${base_mass}" />
+      <origin xyz="0 0 0" />
+      <inertia  ixx="${base_mass*(3*base_radius*base_radius+base_height*base_height)/12}" ixy = "0" ixz = "0"
+      iyy="${base_mass*(3*base_radius*base_radius+base_height*base_height)/12}" iyz="0"
+      izz="${base_mass*base_radius*base_radius/2}" />
     </inertial>
-    <collision name='collision'>
-      <geometry>
-        <box size=".4 .2 .1"/>
-      </geometry>
-    </collision>
-    <visual name='chassis_visual'>
-      <origin xyz="0 0 0" rpy=" 0 0 0"/>
-      <geometry>
-        <box size=".4 .2 .1"/>
-      </geometry>
+    <visual>
+        <geometry>
+            <cylinder length="${base_height}" radius="${base_radius}" />
+        </geometry>
     </visual>
-    <collision name='caster_collision'>
-      <origin xyz="-0.15 0 -0.05" rpy=" 0 0 0"/>
-      <geometry>
-        <sphere radius="0.05"/>
-      </geometry>
-      <surface>
-        <friction>
-          <ode>
-            <mu>0</mu>
-            <mu2>0</mu2>
-            <slip1>1.0</slip1>
-            <slip2>1.0</slip2>
-          </ode>
-        </friction>
-      </surface>
-    </collision>
-    <visual name='caster_visual'>
-      <origin xyz="-0.15 0 -0.05" rpy=" 0 0 0"/>
-      <geometry>
-        <sphere radius="0.05"/>
-      </geometry>
-    </visual>
-  </link>
-  <link name="left_wheel">
-    <collision name="collision">
-      <origin xyz="0 0 0" rpy="0 1.5707 1.5707"/>
-      <geometry>
-        <cylinder radius="0.1" length="0.05"/>
-      </geometry>
-    </collision>
-    <visual name="left_wheel_visual">
-      <origin xyz="0 0 0" rpy="0 1.5707 1.5707"/>
-      <geometry>
-        <cylinder radius="0.1" length="0.05"/>
-      </geometry>
-    </visual>
-    <inertial>
-      <origin xyz="0 0 0" rpy="0 1.5707 1.5707"/>
-      <mass value="5"/>
-      <cylinder_inertia m="5" r="0.1" h="0.05"/>
-      <inertia
-        ixx="1.0" ixy="0.0" ixz="0.0"
-        iyy="1.0" iyz="0.0"
-        izz="1.0"/>
-    </inertial>
-  </link>
-  <link name="right_wheel">
-    <collision name="collision">
-      <origin xyz="0 0 0" rpy="0 1.5707 1.5707"/>
-      <geometry>
-        <cylinder radius="0.1" length="0.05"/>
-      </geometry>
-    </collision>
-    <visual name="right_wheel_visual">
-      <origin xyz="0 0 0" rpy="0 1.5707 1.5707"/>
-      <geometry>
-        <cylinder radius="0.1" length="0.05"/>
-      </geometry>
-    </visual>
-    <inertial>
-      <origin xyz="0 0 0" rpy="0 1.5707 1.5707"/>
-      <mass value="5"/>
-      <cylinder_inertia m="5" r="0.1" h="0.05"/>
-      <inertia
-        ixx="1.0" ixy="0.0" ixz="0.0"
-        iyy="1.0" iyz="0.0"
-        izz="1.0"/>
-    </inertial>
-  </link>
-  <joint type="continuous" name="left_wheel_hinge">
-    <origin xyz="0.1 0.15 0" rpy="0 0 0"/>
-    <child link="left_wheel"/>
-    <parent link="chassis"/>
-    <axis xyz="0 1 0" rpy="0 0 0"/>
-    <limit effort="100" velocity="100"/>
-    <joint_properties damping="0.0" friction="0.0"/>
-  </joint>
-  <joint type="continuous" name="right_wheel_hinge">
-    <origin xyz="0.1 -0.15 0" rpy="0 0 0"/>
-    <child link="right_wheel"/>
-    <parent link="chassis"/>
-    <axis xyz="0 1 0" rpy="0 0 0"/>
-    <limit effort="100" velocity="100"/>
-    <joint_properties damping="0.0" friction="0.0"/>
-  </joint>
-  <joint name="hokuyo_joint" type="fixed">
-    <origin xyz=".15 0 .1" rpy="0 0 0"/>
-    <parent link="chassis"/>
-    <child link="hokuyo"/>
-  </joint>
-  <link name="hokuyo">
     <collision>
-      <origin xyz="0 0 0" rpy="0 0 0" />
         <geometry>
-          <box size="0.1 0.1 0.1" />
+            <cylinder length="${base_height}" radius="${base_radius}" />
         </geometry>
     </collision>
-    <visual>
-      <origin xyz="0 0 0" rpy="0 0 0" />
-        <geometry>
-          <box size="0.1 0.1 0.1"/>
-        </geometry>
-    </visual>
-    <inertial>
-      <mass value="1e-5" />
-      <origin xyz="0 0 0" rpy="0 0 0" />
-      <inertia ixx="1e-6" ixy="0" ixz="0" iyy="1e-6" iyz="0" izz="1e-6" />
-    </inertial>
   </link>
-   <transmission name="left_wheel_joint_trans">
-     <type>transmission_interface/SimpleTransmission</type>
-     <joint name="left_wheel_hinge" >
-       <hardwareInterface>hardware_interface/EffortJointInterface</hardwareInterface>
-     </joint>
-     <actuator name="left_wheel_actuator">
-       <hardwareInterface>EffortJointInterface</hardwareInterface>
-       <mechanicalReduction>10</mechanicalReduction>
-     </actuator>
-   </transmission>
-   <transmission name="right_wheel_joint_trans">
-     <type>transmission_interface/SimpleTransmission</type>
-     <joint name="right_wheel_hinge" >
-       <hardwareInterface>hardware_interface/EffortJointInterface</hardwareInterface>
-     </joint>
-     <actuator name="right_wheel_actuator">
-       <hardwareInterface>EffortJointInterface</hardwareInterface>
-       <mechanicalReduction>10</mechanicalReduction>
-     </actuator>
-   </transmission>
 </robot>

Commit message: new robot add caster

File: src/mybot_description/urdf/mybot.xacro (robot description, xacro)
@@ -7,4 +7,10 @@
   <property name="base_radius" value="0.15"/>
   <property name="base_height" value="0.02"/>
+  <property name="caster_height" value="0.04" />
+  <property name="caster_radius" value="0.025" />
+  <property name="caster_mass" value="0.5" />
+  <property name="wheel_mass" value="2.5" />
+  <property name="wheel_radius" value="0.04" />
+  <property name="wheel_height" value="0.02" />
   <link name='chassis'>
     <inertial>
@@ -26,3 +32,91 @@
     </collision>
   </link>
+  <link name="caster_front_link">
+    <visual>
+      <origin xyz="0 0.02 0" />
+      <geometry>
+        <sphere radius="${caster_radius}" />
+      </geometry>
+    </visual>
+    <collision>
+      <geometry>
+        <sphere radius="${caster_radius}" />
+      </geometry>
+      <origin xyz="0 0.02 0" rpy="${M_PI/2} 0 0" />
+    </collision>
+    <inertial>
+      <mass value="${caster_mass}" />
+      <origin xyz="0 0 0" />
+      <inertia ixx="0.001" ixy="0.0" ixz="0.0"
+        iyy="0.001" iyz="0.0"
+        izz="0.001" />
+      </inertial>
+  </link>
+  <link name="caster_back_link">
+    <visual>
+      <origin xyz="0 0.02 0" />
+      <geometry>
+        <sphere radius="${caster_radius}" />
+      </geometry>
+    </visual>
+    <collision>
+      <geometry>
+        <sphere radius="${caster_radius}" />
+      </geometry>
+      <origin xyz="0 0.02 0" rpy="${M_PI/2} 0 0" />
+    </collision>
+    <inertial>
+      <mass value="${caster_mass}" />
+      <origin xyz="0 0 0" />
+      <inertia ixx="0.001" ixy="0.0" ixz="0.0"
+        iyy="0.001" iyz="0.0"
+        izz="0.001" />
+      </inertial>
+  </link>
+   <joint name="caster_back_joint" type="fixed">
+     <parent link="chassis"/>
+     <child link="caster_back_link"/>
+     <origin xyz="-0.135 0.0 0.009" rpy="${-M_PI/2} 0 0"/>
+   </joint>
+   <joint name="caster_front_joint" type="fixed">
+     <parent link="chassis"/>
+     <child link="caster_front_link"/>
+     <origin xyz="0.115 0.0 0.007" rpy="${-M_PI/2} 0 0"/>
+  </joint>
+  <link name="left_wheel">
+    <visual>
+      <geometry>
+        <cylinder length="${wheel_height}" radius="${wheel_radius}" />
+      </geometry>
+    </visual>
+    <collision>
+      <geometry>
+        <cylinder length="${wheel_height}" radius="${wheel_radius}" />
+      </geometry>
+    </collision>
+    <inertial>
+      <mass value="${wheel_mass}" />
+      <origin xyz="0 0 0" />
+      <inertia  ixx="${wheel_mass*(3*wheel_radius*wheel_radius+wheel_height*wheel_height)/12}" ixy = "0" ixz = "0"
+      iyy="${wheel_mass*(3*wheel_radius*wheel_radius+wheel_height*wheel_height)/12}" iyz="0"
+      izz="${wheel_mass*wheel_radius*wheel_radius/2}" />
+  </link>
+  <link name="right_wheel">
+    <visual>
+      <geometry>
+        <cylinder length="${wheel_height}" radius="${wheel_radius}" />
+      </geometry>
+    </visual>
+    <collision>
+      <geometry>
+        <cylinder length="${wheel_height}" radius="${wheel_radius}" />
+      </geometry>
+    </collision>
+    <inertial>
+      <mass value="${wheel_mass}" />
+      <origin xyz="0 0 0" />
+      <inertia  ixx="${wheel_mass*(3*wheel_radius*wheel_radius+wheel_height*wheel_height)/12}" ixy = "0" ixz = "0"
+      iyy="${wheel_mass*(3*wheel_radius*wheel_radius+wheel_height*wheel_height)/12}" iyz="0"
+      izz="${wheel_mass*wheel_radius*wheel_radius/2}" />
+  </link>
 </robot>

Commit message: first version robot fix error

File: src/mybot_description/urdf/mybot.xacro (robot description, xacro)
@@ -2,121 +2,154 @@
 <robot name="myrobot" xmlns:xacro="http://www.ros.org/wiki/xacro">
   <xacro:include filename="$(find mybot_description)/urdf/mybot.gazebo" />
-  <property name="M_PI" value="3.14159" />
-  <property name="M_PI_2" value="3.14159" />
-  <property name="base_mass" value="5" />
-  <property name="base_radius" value="0.15"/>
-  <property name="base_height" value="0.02"/>
-  <property name="caster_height" value="0.04" />
-  <property name="caster_radius" value="0.025" />
-  <property name="caster_mass" value="0.5" />
-  <property name="wheel_mass" value="2.5" />
-  <property name="wheel_radius" value="0.04" />
-  <property name="wheel_height" value="0.02" />
   <link name='chassis'>
+    <pose>0 0 0.1 0 0 0</pose>
     <inertial>
-      <mass value="${base_mass}" />
-      <origin xyz="0 0 0" />
-      <inertia  ixx="${base_mass*(3*base_radius*base_radius+base_height*base_height)/12}" ixy = "0" ixz = "0"
-      iyy="${base_mass*(3*base_radius*base_radius+base_height*base_height)/12}" iyz="0"
-      izz="${base_mass*base_radius*base_radius/2}" />
+      <mass value="10.0"/>
+      <origin xyz="0.0 0 0.1" rpy=" 0 0 0"/>
+      <inertia
+          ixx="0.5" ixy="0" ixz="0"
+          iyy="1" iyz="0"
+          izz="0.1"
+      />
     </inertial>
+    <collision name='collision'>
+      <geometry>
+        <box size=".4 .2 .1"/>
+      </geometry>
+    </collision>
+    <visual name='chassis_visual'>
+      <origin xyz="0 0 0" rpy=" 0 0 0"/>
+      <geometry>
+        <box size=".4 .2 .1"/>
+      </geometry>
+    </visual>
+    <collision name='caster_collision'>
+      <origin xyz="-0.15 0 -0.05" rpy=" 0 0 0"/>
+      <geometry>
+        <sphere radius="0.05"/>
+      </geometry>
+      <surface>
+        <friction>
+          <ode>
+            <mu>0</mu>
+            <mu2>0</mu2>
+            <slip1>1.0</slip1>
+            <slip2>1.0</slip2>
+          </ode>
+        </friction>
+      </surface>
+    </collision>
+    <visual name='caster_visual'>
+      <origin xyz="-0.15 0 -0.05" rpy=" 0 0 0"/>
+      <geometry>
+        <sphere radius="0.05"/>
+      </geometry>
+    </visual>
+  </link>
+  <link name="left_wheel">
+    <collision name="collision">
+      <origin xyz="0 0 0" rpy="0 1.5707 1.5707"/>
+      <geometry>
+        <cylinder radius="0.1" length="0.05"/>
+      </geometry>
+    </collision>
+    <visual name="left_wheel_visual">
+      <origin xyz="0 0 0" rpy="0 1.5707 1.5707"/>
+      <geometry>
+        <cylinder radius="0.1" length="0.05"/>
+      </geometry>
+    </visual>
+    <inertial>
+      <origin xyz="0 0 0" rpy="0 1.5707 1.5707"/>
+      <mass value="5"/>
+      <cylinder_inertia m="5" r="0.1" h="0.05"/>
+      <inertia
+        ixx="1.0" ixy="0.0" ixz="0.0"
+        iyy="1.0" iyz="0.0"
+        izz="1.0"/>
+    </inertial>
+  </link>
+  <link name="right_wheel">
+    <collision name="collision">
+      <origin xyz="0 0 0" rpy="0 1.5707 1.5707"/>
+      <geometry>
+        <cylinder radius="0.1" length="0.05"/>
+      </geometry>
+    </collision>
+    <visual name="right_wheel_visual">
+      <origin xyz="0 0 0" rpy="0 1.5707 1.5707"/>
+      <geometry>
+        <cylinder radius="0.1" length="0.05"/>
+      </geometry>
+    </visual>
+    <inertial>
+      <origin xyz="0 0 0" rpy="0 1.5707 1.5707"/>
+      <mass value="5"/>
+      <cylinder_inertia m="5" r="0.1" h="0.05"/>
+      <inertia
+        ixx="1.0" ixy="0.0" ixz="0.0"
+        iyy="1.0" iyz="0.0"
+        izz="1.0"/>
+    </inertial>
+  </link>
+  <joint type="continuous" name="left_wheel_hinge">
+    <origin xyz="0.1 0.15 0" rpy="0 0 0"/>
+    <child link="left_wheel"/>
+    <parent link="chassis"/>
+    <axis xyz="0 1 0" rpy="0 0 0"/>
+    <limit effort="100" velocity="100"/>
+    <joint_properties damping="0.0" friction="0.0"/>
+  </joint>
+  <joint type="continuous" name="right_wheel_hinge">
+    <origin xyz="0.1 -0.15 0" rpy="0 0 0"/>
+    <child link="right_wheel"/>
+    <parent link="chassis"/>
+    <axis xyz="0 1 0" rpy="0 0 0"/>
+    <limit effort="100" velocity="100"/>
+    <joint_properties damping="0.0" friction="0.0"/>
+  </joint>
+  <joint name="hokuyo_joint" type="fixed">
+    <origin xyz=".15 0 .1" rpy="0 0 0"/>
+    <parent link="chassis"/>
+    <child link="hokuyo"/>
+  </joint>
+  <link name="hokuyo">
+    <collision>
+      <origin xyz="0 0 0" rpy="0 0 0" />
+        <geometry>
+          <box size="0.1 0.1 0.1" />
+        </geometry>
+    </collision>
     <visual>
+      <origin xyz="0 0 0" rpy="0 0 0" />
         <geometry>
-            <cylinder length="${base_height}" radius="${base_radius}" />
+          <box size="0.1 0.1 0.1"/>
         </geometry>
     </visual>
-    <collision>
-        <geometry>
-            <cylinder length="${base_height}" radius="${base_radius}" />
-        </geometry>
-    </collision>
+    <inertial>
+      <mass value="1e-5" />
+      <origin xyz="0 0 0" rpy="0 0 0" />
+      <inertia ixx="1e-6" ixy="0" ixz="0" iyy="1e-6" iyz="0" izz="1e-6" />
+    </inertial>
   </link>
-  <link name="caster_front_link">
-    <visual>
-      <origin xyz="0 0.02 0" />
-      <geometry>
-        <sphere radius="${caster_radius}" />
-      </geometry>
-    </visual>
-    <collision>
-      <geometry>
-        <sphere radius="${caster_radius}" />
-      </geometry>
-      <origin xyz="0 0.02 0" rpy="${M_PI/2} 0 0" />
-    </collision>
-    <inertial>
-      <mass value="${caster_mass}" />
-      <origin xyz="0 0 0" />
-      <inertia ixx="0.001" ixy="0.0" ixz="0.0"
-        iyy="0.001" iyz="0.0"
-        izz="0.001" />
-      </inertial>
-  </link>
-  <link name="caster_back_link">
-    <visual>
-      <origin xyz="0 0.02 0" />
-      <geometry>
-        <sphere radius="${caster_radius}" />
-      </geometry>
-    </visual>
-    <collision>
-      <geometry>
-        <sphere radius="${caster_radius}" />
-      </geometry>
-      <origin xyz="0 0.02 0" rpy="${M_PI/2} 0 0" />
-    </collision>
-    <inertial>
-      <mass value="${caster_mass}" />
-      <origin xyz="0 0 0" />
-      <inertia ixx="0.001" ixy="0.0" ixz="0.0"
-        iyy="0.001" iyz="0.0"
-        izz="0.001" />
-      </inertial>
-  </link>
-   <joint name="caster_back_joint" type="fixed">
-     <parent link="chassis"/>
-     <child link="caster_back_link"/>
-     <origin xyz="-0.135 0.0 0.009" rpy="${-M_PI/2} 0 0"/>
-   </joint>
-   <joint name="caster_front_joint" type="fixed">
-     <parent link="chassis"/>
-     <child link="caster_front_link"/>
-     <origin xyz="0.115 0.0 0.007" rpy="${-M_PI/2} 0 0"/>
-  </joint>
-  <link name="left_wheel">
-    <visual>
-      <geometry>
-        <cylinder length="${wheel_height}" radius="${wheel_radius}" />
-      </geometry>
-    </visual>
-    <collision>
-      <geometry>
-        <cylinder length="${wheel_height}" radius="${wheel_radius}" />
-      </geometry>
-    </collision>
-    <inertial>
-      <mass value="${wheel_mass}" />
-      <origin xyz="0 0 0" />
-      <inertia  ixx="${wheel_mass*(3*wheel_radius*wheel_radius+wheel_height*wheel_height)/12}" ixy = "0" ixz = "0"
-      iyy="${wheel_mass*(3*wheel_radius*wheel_radius+wheel_height*wheel_height)/12}" iyz="0"
-      izz="${wheel_mass*wheel_radius*wheel_radius/2}" />
-  </link>
-  <link name="right_wheel">
-    <visual>
-      <geometry>
-        <cylinder length="${wheel_height}" radius="${wheel_radius}" />
-      </geometry>
-    </visual>
-    <collision>
-      <geometry>
-        <cylinder length="${wheel_height}" radius="${wheel_radius}" />
-      </geometry>
-    </collision>
-    <inertial>
-      <mass value="${wheel_mass}" />
-      <origin xyz="0 0 0" />
-      <inertia  ixx="${wheel_mass*(3*wheel_radius*wheel_radius+wheel_height*wheel_height)/12}" ixy = "0" ixz = "0"
-      iyy="${wheel_mass*(3*wheel_radius*wheel_radius+wheel_height*wheel_height)/12}" iyz="0"
-      izz="${wheel_mass*wheel_radius*wheel_radius/2}" />
-  </link>
+   <transmission name="left_wheel_joint_trans">
+     <type>transmission_interface/SimpleTransmission</type>
+     <joint name="left_wheel_hinge" >
+       <hardwareInterface>hardware_interface/EffortJointInterface</hardwareInterface>
+     </joint>
+     <actuator name="left_wheel_actuator">
+       <hardwareInterface>EffortJointInterface</hardwareInterface>
+       <mechanicalReduction>10</mechanicalReduction>
+     </actuator>
+   </transmission>
+   <transmission name="right_wheel_joint_trans">
+     <type>transmission_interface/SimpleTransmission</type>
+     <joint name="right_wheel_hinge" >
+       <hardwareInterface>hardware_interface/EffortJointInterface</hardwareInterface>
+     </joint>
+     <actuator name="right_wheel_actuator">
+       <hardwareInterface>EffortJointInterface</hardwareInterface>
+       <mechanicalReduction>10</mechanicalReduction>
+     </actuator>
+   </transmission>
 </robot>

Commit message: can move to goal

File: src/mybot_description/urdf/mybot.xacro (robot description, xacro)
@@ -5,9 +5,9 @@
     <pose>0 0 0.1 0 0 0</pose>
     <inertial>
-      <mass value="10.0"/>
+      <mass value="15.0"/>
       <origin xyz="0.0 0 0.1" rpy=" 0 0 0"/>
       <inertia
-          ixx="0.5" ixy="0" ixz="0"
-          iyy="1" iyz="0"
+          ixx="0.1" ixy="0" ixz="0"
+          iyy="0.1" iyz="0"
           izz="0.1"
       />
@@ -46,4 +46,26 @@
       </geometry>
     </visual>
+    <collision name='caster_front_collision'>
+      <origin xyz="0.15 0 -0.05" rpy=" 0 0 0"/>
+      <geometry>
+        <sphere radius="0.05"/>
+      </geometry>
+      <surface>
+        <friction>
+          <ode>
+            <mu>0</mu>
+            <mu2>0</mu2>
+            <slip1>1.0</slip1>
+            <slip2>1.0</slip2>
+          </ode>
+        </friction>
+      </surface>
+    </collision>
+    <visual name='caster_front_visual'>
+      <origin xyz="0.15 0 -0.05" rpy=" 0 0 0"/>
+      <geometry>
+        <sphere radius="0.05"/>
+      </geometry>
+    </visual>
   </link>
   <link name="left_wheel">
@@ -65,7 +87,7 @@
       <cylinder_inertia m="5" r="0.1" h="0.05"/>
       <inertia
-        ixx="1.0" ixy="0.0" ixz="0.0"
-        iyy="1.0" iyz="0.0"
-        izz="1.0"/>
+        ixx="0.1" ixy="0.0" ixz="0.0"
+        iyy="0.1" iyz="0.0"
+        izz="0.1"/>
     </inertial>
   </link>
@@ -88,24 +110,24 @@
       <cylinder_inertia m="5" r="0.1" h="0.05"/>
       <inertia
-        ixx="1.0" ixy="0.0" ixz="0.0"
-        iyy="1.0" iyz="0.0"
-        izz="1.0"/>
+        ixx="0.1" ixy="0.0" ixz="0.0"
+        iyy="0.1" iyz="0.0"
+        izz="0.1"/>
     </inertial>
   </link>
   <joint type="continuous" name="left_wheel_hinge">
-    <origin xyz="0.1 0.15 0" rpy="0 0 0"/>
+    <origin xyz="0 0.15 0" rpy="0 0 0"/>
     <child link="left_wheel"/>
     <parent link="chassis"/>
     <axis xyz="0 1 0" rpy="0 0 0"/>
-    <limit effort="100" velocity="100"/>
-    <joint_properties damping="0.0" friction="0.0"/>
+    <limit effort="10000" velocity="1000"/>
+    <joint_properties damping="1.0" friction="1.0"/>
   </joint>
   <joint type="continuous" name="right_wheel_hinge">
-    <origin xyz="0.1 -0.15 0" rpy="0 0 0"/>
+    <origin xyz="0 -0.15 0" rpy="0 0 0"/>
     <child link="right_wheel"/>
     <parent link="chassis"/>
     <axis xyz="0 1 0" rpy="0 0 0"/>
-    <limit effort="100" velocity="100"/>
-    <joint_properties damping="0.0" friction="0.0"/>
+    <limit effort="10000" velocity="1000"/>
+    <joint_properties damping="1.0" friction="1.0"/>
   </joint>
   <joint name="hokuyo_joint" type="fixed">
